Commit message: added environment variable reference for passing parameter into .gazebo.xacro

File: urdf/turtlebot3_waffle.gazebo.xacro (robot description, xacro)
@@ -4,4 +4,5 @@
   <xacro:arg name="camera_visual" default="false"/>
   <xacro:arg name="imu_visual"    default="false"/>
+  <xacro:property name="laser_range_val" value="$(env LASER_RANGE_VAL)"/>
   <gazebo reference="base_link">
     <material>Gazebo/DarkGrey</material>
@@ -119,5 +120,5 @@
         <range>
           <min>0.120</min>
-          <max>1.35</max>
+          <max>${laser_range_val}</max>
           <resolution>0.015</resolution>
         </range>

Commit message: commit

File: urdf/turtlebot3_waffle.gazebo.xacro (robot description, xacro)
@@ -5,4 +5,6 @@
   <xacro:arg name="imu_visual"    default="false"/>
   <xacro:property name="laser_range_val" value="$(env LASER_RANGE_VAL)"/>
+  <xacro:property name="laser_update_rate" value="$(env LASER_UPDATE_RATE)"/>
+  <xacro:property name="imu_update_rate" value="$(env IMU_UPDATE_RATE)"/>
   <gazebo reference="base_link">
     <material>Gazebo/DarkGrey</material>

Commit message: clean up files, added Laser and IMU "noise" parameters with list of values. Current Main_Director script will itterate over ALL paramters

File: urdf/turtlebot3_waffle.gazebo.xacro (robot description, xacro)
@@ -5,6 +5,7 @@
   <xacro:arg name="imu_visual"    default="false"/>
   <xacro:property name="laser_range_val" value="$(env LASER_RANGE_VAL)"/>
-  <xacro:property name="laser_update_rate" value="$(env LASER_UPDATE_RATE)"/>
-  <xacro:property name="imu_update_rate" value="$(env IMU_UPDATE_RATE)"/>
+  <xacro:property name="laser_noise_stddev" value="$(env LASER_NOISE_STDDEV)"/>
+  <xacro:property name="imu_gyro_noise_stddev" value="$(env IMU_GYRO_NOISE_STDDEV)"/>
+  <xacro:property name="imu_accel_noise_stddev" value="$(env IMU_ACCEL_NOISE_STDDEV)"/>
   <gazebo reference="base_link">
     <material>Gazebo/DarkGrey</material>
@@ -91,5 +92,5 @@
           <rate>
             <mean>0.0</mean>
-            <stddev>2e-4</stddev>
+            <stddev>${imu_gyro_noise_stddev}</stddev>
             <bias_mean>0.0000075</bias_mean>
             <bias_stddev>0.0000008</bias_stddev>
@@ -97,5 +98,5 @@
           <accel>
             <mean>0.0</mean>
-            <stddev>1.7e-2</stddev>
+            <stddev>${imu_accel_noise_stddev}</stddev>
             <bias_mean>0.1</bias_mean>
             <bias_stddev>0.001</bias_stddev>
@@ -128,5 +129,5 @@
           <type>gaussian</type>
           <mean>0.0</mean>
-          <stddev>0.01</stddev>
+          <stddev>${laser_noise_stddev}</stddev>
         </noise>
       </ray>
